File: kicad/recovery.kicad_pcb (KiCad board)
At the start: 2 copper layers, 84.1 x 61.7 mm, 50 parts, among them J1 Bus_PCI_Express_x1, J2 wago 2060-452/998-404, J3 wago 2060-452/998-404, J4 Conn_01x04, J5 Conn_01x02_Pin, J6 USB_C_Receptacle_USB2.0_16P, Q1 SI7232DN-T1-GE3, U2 RP2040, U4 W25Q128JVP, U9 MCP25625T-E/ML, X1 RP2040 Crystal, Y2 X322516MLB4SI

Commit message: finish routing
Parts:
- moved J4 5.18 mm to (124.4, 92.7)
- moved J2 1.10 mm to (125.5, 113.4)
Connections:
- U2 pad 39: sense_d -> sense_m
- U2 pad 40: sense_m -> sense_d
Routing:
- net sense_d: track 1.09 -> 34.3 mm, vias 0 -> 2
- net sense_m: track 0.98 -> 31.2 mm, vias 0 -> 2
- net +3.3V: track 105.3 -> 132.6 mm, vias 7 -> 10
- net /SWCLK: track 29.3 -> 24.0 mm
- net /SWD: track 27.0 -> 23.8 mm
- net v_lipo: track 122.1 -> 124.1 mm, vias 0 -> 3
- net +5V: track 41.2 -> 43.2 mm, vias 1 -> 4
- net GND: track 16.3 -> 17.7 mm, vias 96 -> 182
- net +1V1: track 15.0 -> 14.4 mm
