File: kicad/recovery.kicad_pcb (KiCad board)
At the start: 2 copper layers, 84.1 x 61.7 mm, 50 parts, among them J1 Bus_PCI_Express_x1, J2 wago 2060-452/998-404, J3 wago 2060-452/998-404, J4 Conn_01x04, J5 Conn_01x02_Pin, J6 USB_C_Receptacle_USB2.0_16P, Q1 SI7232DN-T1-GE3, U2 RP2040, U4 W25Q128JVP, U9 MCP25625T-E/ML, X1 RP2040 Crystal, Y2 X322516MLB4SI

Commit message: final gerber export
Parts:
- moved C1 12.2 mm to (171.3, 102.2), turned to 0 degrees
- moved J3 2.34 mm to (167.8, 113.4)
- moved J2 0.44 mm to (125.1, 113.4)
Routing:
- net v_lipo: track 124.1 -> 119.1 mm
- net Net-(J3-1_1): track 24.5 -> 25.5 mm
- net Net-(J2-1_1): track 92.9 -> 92.3 mm
- net GND: vias 182 -> 178
Other:
- board text added: "+-"
