File: kicad/recovery.kicad_sch (KiCad schematic)
At the start: 50 parts, among them J1 Bus_PCI_Express_x1, J2 wago 2060-452/998-404, J3 wago 2060-452/998-404, J4 Conn_01x04, J5 Conn_01x02_Pin, J6 USB_C_Receptacle_USB2.0_16P, Q1 SI7232DN-T1-GE3, U2 RP2040, U4 W25Q128JVP, U9 MCP25625T-E/ML, X1 RP2040 Crystal, Y2 X322516MLB4SI

Commit message: final gerber export
Parts:
- J1: now not fitted

Commit message: Feat: Added load switch, PWM level shifters, ADC and buffer circuitry, connectors and solenod driver to schematic
Fix: Reorganized schematic to be readable, modified parachute circuit to utilize 5V.
Parts:
- added C2, C3: 100pF, PCM_JLCPCB:C_0402, symbol PCM_JLCPCB-Capacitors:0402,100pF
- added C21, C28: 1uF, PCM_JLCPCB:C_0603, symbol PCM_JLCPCB-Capacitors:0603,1uF
- added C29, C30: 100nF, PCM_JLCPCB:C_0402, symbol PCM_JLCPCB-Capacitors:0402,100nF
- added C31: 22nF, PCM_JLCPCB:C_0603, symbol PCM_JLCPCB-Capacitors:0603,22nF
- added CN1: S08B-PASK-2(LF)(SN), easyeda2kicad:CONN-TH_S08B-PASK-2, symbol easyeda2kicad:S08B-PASK-2(LF)(SN)
- added D2: SS210, PCM_JLCPCB:D_SMA, symbol PCM_JLCPCB-Diodes:Schottky,SS210
- added Q2, Q3: AO3400A, PCM_JLCPCB:Q_SOT-23, symbol PCM_JLCPCB-Transistors:NMOS,AO3400A
- added R1, R9: 100Ω, PCM_JLCPCB:R_0402, symbol PCM_JLCPCB-Resistors:0402,100Ω
- added R10: 300Ω, PCM_JLCPCB:R_0603, symbol PCM_JLCPCB-Resistors:0603,300Ω
- added R11: 27Ω, PCM_JLCPCB:R_0603, symbol PCM_JLCPCB-Resistors:0603,27Ω
- added R13, R14, R16, R17, R19, R24: 5.1kΩ, PCM_JLCPCB:R_0603, symbol PCM_JLCPCB-Resistors:0603,5.1kΩ
- added R15, R18: 120Ω, PCM_JLCPCB:R_0603, symbol PCM_JLCPCB-Resistors:0603,120Ω
- added R25, R26: 10kΩ, PCM_JLCPCB:R_0402, symbol PCM_JLCPCB-Resistors:0402,10kΩ
- added R27, R28: 10Ω, PCM_JLCPCB:R_0603, symbol PCM_JLCPCB-Resistors:0603,10Ω
- added R29, R34: 5.1Ω, PCM_JLCPCB:R_0603, symbol PCM_JLCPCB-Resistors:0603,5.1Ω
- added R5, R7: 100kΩ, PCM_JLCPCB:R_0402, symbol PCM_JLCPCB-Resistors:0402,100kΩ
- added R6, R8: 33kΩ, PCM_JLCPCB:R_0402, symbol PCM_JLCPCB-Resistors:0402,33kΩ
- added U1: MCP6002T-I/SN, easyeda2kicad:SOIC-8_L4.9-W3.9-P1.27-LS6.0-BL, symbol easyeda2kicad:MCP6002T-I_SN
- added U12, U13: S03B-PASK-2, easyeda2kicad:CONN-TH_S03B-PASK-2-LF-SN, symbol easyeda2kicad:S03B-PASK-2(LF)(SN)
- added U5: TPS22976DPUR, easyeda2kicad:WSON-14_L3.0-W2.0-P0.40-BL-EP-1, symbol easyeda2kicad:TPS22976DPUR
- added U6: GAQY252G3S, easyeda2kicad:SOP-4_L4.3-W4.4-P2.54-LS7.0-BL, symbol easyeda2kicad:GAQY252G3S
Connections:
- net +3.3V: now also R10.1, R15.1, R16.2, R17.2, R18.1, R25.2, R26.2, U1.8 (VDD)
- net +5V: now also C1.1, J2.3 (2_1), J2.4 (2_2), J3.3 (2_1), J3.4 (2_2)
- net CANSTBY: no longer U2.38 (GPIO26_ADC0)
- net GND: now also C2.2, C21.2, C28.2, C29.2, C3.2, C30.2, CN1.1, CN1.2, CN1.3, D2.1, R11.2, R13.1, R14.1, R16.1, R17.1, R27.2, R28.2, R6.2, R8.2, U1.4 (-VSS), U13.1, U5.11 (GND), U5.15 (EP), U6.2, U6.3
- net sense_d: now also U2.39 (GPIO27_ADC1); no longer U2.40 (GPIO28_ADC2)
- net sense_m: now also U2.38 (GPIO26_ADC0); no longer U2.39 (GPIO27_ADC1)
- net v_lipo: no longer C1.1, J2.3 (2_1), J2.4 (2_2), J3.3 (2_1), J3.4 (2_2)
- net at Q1.7, Q1.8, R32.2: now also R34.1; no longer J2.1 (1_1), J2.2 (1_2)
- net at Q1.5, Q1.6, R22.2: now also R29.1; no longer J3.1 (1_1), J3.2 (1_2)
- net PT_2: now reaches U2.41 (GPIO29_ADC3)
- net PT_2: now also C3.1, R9.2
- new net: Q2.1 (G), R15.2
- new net: C31.2, R11.1
- new net: R7.2, R8.1, U1.5 (+INB)
- new net: R10.2, U6.1
- new net: Q3.1 (G), R18.2
- new net: R5.2, R6.1, U1.3 (+INA)
- new net: J2.1 (1_1), J2.2 (1_2), R34.2
- new net: J3.1 (1_1), J3.2 (1_2), R29.2
- new net +24V: C31.1, D2.2, U12.3, U6.4
- new net +5V_Servo: C21.1, C28.1, R19.2, R24.2, U5.1 (VIN1), U5.2 (VIN1), U5.4 (VBIAS), U5.6 (VIN2), U5.7 (VIN2)
- new net 3.3V_PWM1: Q2.2 (S), R25.1
- new net 3.3V_PWM2: Q3.2 (S), R26.1
- new net 5V_PWM1: Q2.3 (D), R24.1, U12.2
- new net 5V_PWM2: Q3.3 (D), R19.1, U12.1
- new net AIN_0IN: U13.2
- new net AIN_1IN: U13.3
- new net OUTA: R1.2, U1.1 (OUTA), U1.2 (-INA)
- new net OUTB: R9.1, U1.6 (-INB), U1.7 (OUTB)
- new net PT_1: C2.1, R1.1, U2.40 (GPIO28_ADC2)
- new net PT_IN1: R5.1
- new net PT_IN2: R7.1
- new net SERVO_ON1: R13.2, U5.3 (ON1)
- new net SERVO_ON2: R14.2, U5.5 (ON2)
- new net SERVO_PWR1: C29.1, CN1.7, R27.1, U5.13 (VOUT1), U5.14 (VOUT1)
- new net SERVO_PWR2: C30.1, CN1.8, R28.1, U5.8 (VOUT2), U5.9 (VOUT2)
- no-connect marks 34 -> 35
Other:
- note added: "5V/800mA - 1R - 0.015 RDSon = 5.235 R"
- note added: "ADC"
- note added: "CONNECTORS"
- note added: "PWM LEVEL SHIFTER"
- note added: "RP2040"
- note added: "SERVO PWR SWITCH"
- note added: "SOLENOID DRIVER"
- note added: "talk to zeulewan abt the 5.1 ohm, either i figure out constant current source or we use big ass smd resistor"
- note removed: "Make sure R3 and R4 are close to RP2040"
- moved on the sheet: C1, C10, C11, C206, C207, C208, C209, C210, C211, C212, C213, C214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
